Commit message: edit: xacro figure

File: ros2_ws/src/capstone/description/face.xacro (robot description, xacro)
@@ -8,21 +8,21 @@
     <link name="face_link">
         <visual>
-            <origin xyz="0 0.05 0.01" rpy="0 ${pi/2} 0"/>
+            <origin xyz="0 0.08 0.02" rpy="0 ${pi/2} 0"/>
             <geometry>
-                <cylinder radius="0.01" length="0.002"/>
+                <cylinder radius="0.025" length="0.003"/>
             </geometry>
             <material name="black"/>
         </visual>
         <visual>
-            <origin xyz="0 -0.05 0.01" rpy="0 ${pi/2} 0"/>
+            <origin xyz="0 -0.08 0.02" rpy="0 ${pi/2} 0"/>
             <geometry>
-                <cylinder radius="0.01" length="0.002"/>
+                <cylinder radius="0.025" length="0.003"/>
             </geometry>
             <material name="black"/>
         </visual>
         <visual>
-            <origin xyz="-0.011 0 -0.00" rpy="0 ${1.5} 0"/>
+            <origin xyz="-0.011 0 -0.05" rpy="0 ${1.5} 0"/>
             <geometry>
-                <cylinder radius="0.05" length="0.02"/>
+                <cylinder radius="0.045" length="0.0225"/>
             </geometry>
             <material name="red"/>

File: ros2_ws/src/capstone/description/lidar.xacro (robot description, xacro)
@@ -4,17 +4,38 @@
         <parent link="chassis"/>
         <child link="laser_frame"/>
-        <origin xyz="0.162 0 0.514" rpy="0 0 0"/>
+        <origin xyz="0.191 0 0.463" rpy="0 0 0"/>
     </joint>
     <link name="laser_frame">
         <visual>
             <geometry>
-                <cylinder radius="0.05" length="0.04"/>
+                <cylinder radius="0.043" length="0.029"/>
             </geometry>
             <material name="purple"/>
         </visual>
         <visual>
-            <origin xyz="0 0 -0.05"/>
+            <origin xyz="0.028 0.020 -0.05"/>
             <geometry>
-                <cylinder radius="0.01" length="0.1"/>
+                <cylinder radius="0.005" length="0.08"/>
+            </geometry>
+            <material name="purple"/>
+        </visual>
+        <visual>
+            <origin xyz="0.028 -0.020 -0.05"/>
+            <geometry>
+                <cylinder radius="0.005" length="0.08"/>
+            </geometry>
+            <material name="purple"/>
+        </visual>
+        <visual>
+            <origin xyz="-0.028 0.020 -0.05"/>
+            <geometry>
+                <cylinder radius="0.005" length="0.08"/>
+            </geometry>
+            <material name="purple"/>
+        </visual>
+        <visual>
+            <origin xyz="-0.028 -0.020 -0.05"/>
+            <geometry>
+                <cylinder radius="0.005" length="0.08"/>
             </geometry>
             <material name="purple"/>
@@ -22,8 +43,8 @@
         <collision>
             <geometry>
-                <cylinder radius="0.05" length="0.04"/>
+                <cylinder radius="0.033" length="0.029"/>
             </geometry>
         </collision>
-        <xacro:inertial_cylinder mass="0.1" length="0.04" radius="0.05">
+        <xacro:inertial_cylinder mass="0.1" length="0.029" radius="0.033">
             <origin xyz="0 0 0" rpy="0 0 0"/>
         </xacro:inertial_cylinder>

File: ros2_ws/src/capstone/description/robot.urdf.xacro (robot description, xacro)
@@ -12,4 +12,4 @@
     <xacro:include filename="lidar.xacro" />
     <!-- <xacro:include filename="odometry.xacro" /> -->
-    <!-- <xacro:include filename="face.xacro" /> -->
+    <xacro:include filename="face.xacro" />
 </robot>

File: ros2_ws/src/capstone/description/robot_core.xacro (robot description, xacro)
@@ -2,17 +2,17 @@
 <robot xmlns:xacro="http://www.ros.org/wiki/xacro" >
     <xacro:include filename="inertial_macros.xacro"/>
-    <xacro:property name="chassis_length" value="0.335"/>
-    <xacro:property name="chassis_width" value="0.265"/>
-    <xacro:property name="chassis_height" value="0.482"/> <!-- 0.138 -->
-    <xacro:property name="chassis_mass" value="1.0"/>
-    <xacro:property name="wheel_radius" value="0.066"/> <!-- 0.066 -->
-    <xacro:property name="wheel_thickness" value="0.036"/> <!-- 0.026 -->
+    <xacro:property name="chassis_length" value="0.361"/> <!-- 0.335 -->
+    <xacro:property name="chassis_width" value="0.351"/> <!-- 0.261 -->
+    <xacro:property name="chassis_height" value="0.409"/> <!-- 0.482 <- 0.138 -->
+    <xacro:property name="chassis_mass" value="10.0"/> <!-- 1.0 -->
+    <xacro:property name="wheel_radius" value="0.033"/> <!-- 0.066 -->
+    <xacro:property name="wheel_thickness" value="0.026"/> <!-- 0.026 -->
     <xacro:property name="wheel_mass" value="0.05"/>
-    <xacro:property name="wheel_offset_x" value="0.226"/>
-    <xacro:property name="wheel_offset_y" value="0.1485"/>
-    <xacro:property name="wheel_offset_z" value="0.01"/>
-    <xacro:property name="caster_wheel_radius" value="0.02"/> <!-- 0.01 -->
+    <xacro:property name="wheel_offset_x" value="0.261"/>
+    <xacro:property name="wheel_offset_y" value="0.1776"/>
+    <xacro:property name="wheel_offset_z" value="0.0185"/>
+    <xacro:property name="caster_wheel_radius" value="0.014"/> <!-- 0.2 <- 0.01 -->
     <xacro:property name="caster_wheel_mass" value="0.01"/>
-    <xacro:property name="caster_wheel_offset_x" value="0.075"/>
+    <xacro:property name="caster_wheel_offset_x" value="0.089"/>
     <xacro:property name="caster_wheel_offset_z" value="${wheel_offset_z - wheel_radius + caster_wheel_radius}"/>
     <material name="white">
@@ -68,5 +68,5 @@
             </geometry>
         </collision>
-        <xacro:inertial_box mass="0.5" x="${chassis_length}" y="${chassis_width}" z="${chassis_height}">
+        <xacro:inertial_box mass="8.5" x="${chassis_length}" y="${chassis_width}" z="${chassis_height}">
             <origin xyz="${chassis_length/2} 0 ${chassis_height/2}" rpy="0 0 0"/>
         </xacro:inertial_box>

File: ros2_ws/src/capstone/description/ros2_control.xacro (robot description, xacro)
@@ -19,6 +19,6 @@
             <joint name="left_wheel_joint">
                 <command_interface name="velocity">
-                    <param name="min">-10</param>
-                    <param name="max">10</param>
+                    <param name="min">-5</param>
+                    <param name="max">5</param>
                 </command_interface>
                 <state_interface name="velocity"/>
@@ -27,6 +27,6 @@
             <joint name="right_wheel_joint">
                 <command_interface name="velocity">
-                    <param name="min">-10</param>
-                    <param name="max">10</param>
+                    <param name="min">-5</param>
+                    <param name="max">5</param>
                 </command_interface>
                 <state_interface name="velocity"/>
